File: PCB/motor_controller.kicad_sch (KiCad schematic)
At the start: 6 parts, among them J2 Motor1, J3 Motor2, U3 TB6612FNG

Commit message: PCB version to fab
Parts:
- removed C4: 10uF, Capacitor_THT:CP_Radial_D5.0mm_P2.00mm, symbol Device:C_Polarized
- added C1: 10u, Capacitor_SMD:C_0805_2012Metric_Pad1.18x1.45mm_HandSolder, symbol Device:C
- C2, C3: footprint Capacitor_SMD:C_0603_1608Metric_Pad1.08x0.95mm_HandSolder -> Capacitor_SMD:C_0805_2012Metric_Pad1.18x1.45mm_HandSolder
Connections:
- net GND: now also C1.2
- net Vs: now also C1.1
Changed lines of the file:
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@@
+    )
+  )
+  (symbol (lib_id "Device:C") (at 161.29 59.69 90) (unit 1)
+    (in_bom yes) (on_board yes) (dnp no) (fields_autoplaced)
+    (property "Reference" "C1" (at 161.29 52.07 90)
+      (effects (font (size 1.27 1.27)))
+    )
+    (property "Value" "10u" (at 161.29 54.61 90)
+      (effects (font (size 1.27 1.27)))
+    )
+    (property "Footprint" "Capacitor_SMD:C_0805_2012Metric_Pad1.18x1.45mm_HandSolder" (at 165.1 58.7248 0)
+      (effects (font (size 1.27 1.27)) hide)
+    )
+    (property "Datasheet" "~" (at 161.29 59.69 0)
+      (effects (font (size 1.27 1.27)) hide)
+    )
+    (pin "1")
+    (pin "2")
+    (instances
+      (project "ml_robot"
+        (path "/e63e39d7-6ac0-4ffd-8aa3-1841a4541b55/adf16a2c-a27f-43bb-855c-69d07172e297"
+          (reference "C1") (unit 1)
+        )
+      )
     )
   )
@@
       (effects (font (size 1.27 1.27)))
     )
-    (property "Footprint" "Capacitor_SMD:C_0603_1608Metric_Pad1.08x0.95mm_HandSolder" (at 165.1 52.3748 0)
+    (property "Footprint" "Capacitor_SMD:C_0805_2012Metric_Pad1.18x1.45mm_HandSolder" (at 165.1 52.3748 0)
       (effects (font (size 1.27 1.27)) hide)
     )
@@
         (path "/e63e39d7-6ac0-4ffd-8aa3-1841a4541b55/adf16a2c-a27f-43bb-855c-69d07172e297"
           (reference "J3") (unit 1)
-        )
-      )
-    )
-  )
-  (symbol (lib_id "Device:C_Polarized") (at 161.29 59.69 90) (unit 1)
-    (in_bom yes) (on_board yes) (dnp no)
-    (property "Reference" "C4" (at 165.1 62.23 90)
-      (effects (font (size 1.27 1.27)))
-    )
-    (property "Value" "10uF" (at 165.1 64.77 90)
-      (effects (font (size 1.27 1.27)))
-    )
-    (property "Footprint" "Capacitor_THT:CP_Radial_D5.0mm_P2.00mm" (at 165.1 58.7248 0)
-      (effects (font (size 1.27 1.27)) hide)
-    )
-    (property "Datasheet" "~" (at 161.29 59.69 0)
-      (effects (font (size 1.27 1.27)) hide)
-    )
-    (pin "1")
-    (pin "2")
-    (instances
-      (project "ml_robot"
-        (path "/e63e39d7-6ac0-4ffd-8aa3-1841a4541b55/adf16a2c-a27f-43bb-855c-69d07172e297"
-          (reference "C4") (unit 1)
         )
       )
@@
       (effects (font (size 1.27 1.27)))
     )
-    (property "Footprint" "Capacitor_SMD:C_0603_1608Metric_Pad1.08x0.95mm_HandSolder" (at 124.46 67.0052 0)
+    (property "Footprint" "Capacitor_SMD:C_0805_2012Metric_Pad1.18x1.45mm_HandSolder" (at 124.46 67.0052 0)
       (effects (font (size 1.27 1.27)) hide)
     )
